File: inmoov/pcb/shield_jambes/shield_jambes.kicad_pcb (KiCad board)
At the start: 2 copper layers, 101.6 x 53.3 mm, 25 parts, among them J1 Barrette Mega, J10 HX711 n°0, J11 HX711 n°1, J12 HX711 n°2, J13 HX711 n°3, J14 HX711 n°4, J15 HX711 n°5, J16 HX711 n°6, J17 HX711 n°7, J2 Barrette Mega, J20 BNO085, J21 Bus servos, J22 Arret urgence, J3 Barrette Mega, J4 Barrette Mega

Commit message: Ajoute la carte servos 16 voies et le HAT capteurs (DOMOKAMI CONNECT)
- pcb/common/pcbtools.py : outils communs (placement, plans de cuivre,
  routage Freerouting, vias de couture, DRC, Gerber, fichiers JLCPCB)
- pcb/carte_servos : PCA9685 + INA226 + fusible ATO + bornier 24 A,
  16 sorties servo sur plans de cuivre, ponts d'adresse A/B/C ; DRC 0/0
- pcb/hat_capteurs : HAT Raspberry Pi 5 (spécification officielle),
  3 ADS1115 0x48/0x49/0x4A, 10 entrées FSR, 3 sorties I2C ; DRC 0/0
- titre « DOMOKAMI CONNECT » sur les 3 cartes (shield jambes régénéré)
- notices LISEZMOI, aperçus, tests des réseaux et des adresses,
  README et manuel mis à jour

Co-Authored-By: Claude Opus 5.5 <noreply@anthropic.com>
Claude-Session: https://claude.ai/code/session_01KYEqXZtai4eeCvWZwFamok
Other:
- board text added: "DOMOKAMI CONNECT"
- board text added: "shield jambes v1"
- board text removed: "InMoov · shield jambes v1"
